Commit message: feat : made the robot more realistic

File: botzilla_Workspace/src/botzilla_bringup/description/botzilla_qbot.urdf (robot description, URDF)
Before this commit: robot botzilla_qbot, 10 links, 9 joints
Links:
- added link camera_link_optical
Joints:
- added joint camera_optical_joint: type fixed, parent camera_link, child camera_link_optical, origin xyz=0 0 0 rpy=-1.570796 0 -1.570796
- joint camera_joint: origin xyz=0.15 0 0.07 rpy=0 0 0 -> xyz=0.0 0 0.19 rpy=0 0 0
- joint laser_joint: origin xyz=0.0 0.0 0.12 rpy=0 0 0 -> xyz=0.0 0.0 0.24 rpy=0 0 0

Commit message: fix : map ghosting issue

File: botzilla_Workspace/src/botzilla_bringup/description/botzilla_qbot.urdf (robot description, URDF)
Before this commit: robot botzilla_qbot, 11 links, 10 joints
Links:
- added link imu_link, mass 0.01
Joints:
- added joint imu_joint: type fixed, parent base_link, child imu_link, origin xyz=0 0 0 rpy=0 0 0
